Commit message: updates to model

File: vector_common/vector_description/urdf/accessories.urdf.xacro (robot description, xacro)
@@ -27,6 +27,6 @@
         <link name="sic_imu_frame"/>
         <joint name="sic_imu_joint" type="fixed">
-            <origin xyz="0.07475 0.07136 0.24556" rpy="${M_PI} 0 0" />
-            <parent link="$(optenv VECTOR_PARENT_LINK base_chassis_link)" />
+            <origin xyz="0.0326421 0.0899448 0.0082008" rpy="${M_PI} 0 ${M_PI/2}" />
+            <parent link="$(optenv MOVO_PARENT_LINK base_chassis_link)" />
             <child link="sic_imu_frame" />
         </joint>
@@ -36,5 +36,5 @@
                 <updateRate>50.0</updateRate>
                 <bodyName>sic_imu_frame</bodyName>
-                <topicName>/vector/feedback/sic_imu</topicName>
+                <topicName>/movo/feedback/sic_imu</topicName>
                 <accelDrift>0.0005 0.0005 0.0005</accelDrift>
                 <accelGaussianNoise>0.0005 0.0005 0.0005</accelGaussianNoise>
@@ -46,8 +46,8 @@
         </gazebo>
         <xacro:sick_tim laser_prefix="$(optenv LASER1_PREFIX base)" parent="$(optenv VECTOR_PARENT_LINK base_chassis_link)">
-            <origin xyz="$(optenv LASER1_XYZ 0.35 0 0.2)" rpy="$(optenv LASER1_RPY 3.14159 0 0)" />
+            <origin xyz="$(optenv LASER1_XYZ 0.3075 0 0.1439106)" rpy="$(optenv LASER1_RPY 3.14159 0 0)" />
         </xacro:sick_tim>
         <xacro:sick_tim laser_prefix="$(optenv LASER2_PREFIX base)" parent="$(optenv VECTOR_PARENT_LINK base_chassis_link)">
-            <origin xyz="$(optenv LASER2_XYZ 0.35 0 0.2)" rpy="$(optenv LASER2_RPY 3.14159 0 0)" />
+            <origin xyz="$(optenv LASER2_XYZ -0.3075 0 0.1439106)" rpy="$(optenv LASER2_RPY 3.14159 0 3.14159)" />
         </xacro:sick_tim>
     </xacro:macro>

File: vector_common/vector_description/urdf/vector_components/vector_base.urdf.xacro (robot description, xacro)
@@ -45,5 +45,5 @@
             <collision>
 				<geometry>
-					<mesh filename="package://movo_description/meshes/movo_components/collision/vector_base_collision.stl" />
+					<mesh filename="package://vector_description/meshes/vector_components/collision/vector_base_collision.stl" />
 				</geometry>
 			</collision>
@@ -51,5 +51,5 @@
 				<origin xyz="0 0 0" rpy="0 0 0" />
 				<geometry>
-					<mesh filename="package://movo_description/meshes/vector_components/visual/vector_base.dae" />
+					<mesh filename="package://vector_description/meshes/vector_components/visual/vector_base.dae" />
 				</geometry>
 			</visual>
@@ -73,5 +73,5 @@
             <collision>
 				<geometry>
-					<mesh filename="package://movo_description/meshes/movo_components/collision/std_payload_plate_collision.stl" />
+					<mesh filename="package://vector_description/meshes/vector_components/collision/std_payload_plate_collision.stl" />
 				</geometry>
 			</collision>
@@ -79,5 +79,5 @@
 				<origin xyz="0 0 0" rpy="0 0 0" />
 				<geometry>
-					<mesh filename="package://movo_description/meshes/vector_components/visual/std_payload_plate.dae" />
+					<mesh filename="package://vector_description/meshes/vector_components/visual/std_payload_plate.dae" />
 				</geometry>
 			</visual>

Commit message: some fixes from robot integration

File: vector_common/vector_description/urdf/accessories.urdf.xacro (robot description, xacro)
@@ -28,5 +28,5 @@
         <joint name="sic_imu_joint" type="fixed">
             <origin xyz="0.0326421 0.0899448 0.0082008" rpy="${M_PI} 0 ${M_PI/2}" />
-            <parent link="$(optenv MOVO_PARENT_LINK base_chassis_link)" />
+            <parent link="base_chassis_link" />
             <child link="sic_imu_frame" />
         </joint>
@@ -45,8 +45,8 @@
             </plugin>
         </gazebo>
-        <xacro:sick_tim laser_prefix="$(optenv LASER1_PREFIX base)" parent="$(optenv VECTOR_PARENT_LINK base_chassis_link)">
+        <xacro:sick_tim laser_prefix="front" parent="base_chassis_link">
             <origin xyz="$(optenv LASER1_XYZ 0.3075 0 0.1439106)" rpy="$(optenv LASER1_RPY 3.14159 0 0)" />
         </xacro:sick_tim>
-        <xacro:sick_tim laser_prefix="$(optenv LASER2_PREFIX base)" parent="$(optenv VECTOR_PARENT_LINK base_chassis_link)">
+        <xacro:sick_tim laser_prefix="rear" parent="base_chassis_link">
             <origin xyz="$(optenv LASER2_XYZ -0.3075 0 0.1439106)" rpy="$(optenv LASER2_RPY 3.14159 0 3.14159)" />
         </xacro:sick_tim>

Commit message: update for kinetic

File: vector_common/vector_description/urdf/accessories.urdf.xacro (robot description, xacro)
@@ -23,5 +23,5 @@
 <robot name="vector_accessories" xmlns:xacro="http://ros.org/wiki/xacro">
     <xacro:include filename="$(find vector_description)/urdf/sensors/sick_tim.urdf.xacro"/>
-    <property name="M_PI" value="3.14159"/>
+    <xacro:property name="M_PI" value="3.14159"/>
     <xacro:macro name="vector_accessories">
         <link name="sic_imu_frame"/>

File: vector_common/vector_description/urdf/vector.urdf.xacro (robot description, xacro)
@@ -35,8 +35,8 @@
                 <odometryTopic>/vector/odometry/local_filtered</odometryTopic>
                 <odometryFrame>odom</odometryFrame>
-                <odometryRate>30.0</odometryRate>
+                <odometryRate>100.0</odometryRate>
                 <robotBaseFrame>base_link</robotBaseFrame>
                 <publishOdometryTf>1</publishOdometryTf>
-                <yaw_velocity_p_gain>100.0</yaw_velocity_p_gain>
+                <yaw_velocity_p_gain>500.0</yaw_velocity_p_gain>
                 <x_velocity_p_gain>10000.0</x_velocity_p_gain>
                 <y_velocity_p_gain>10000.0</y_velocity_p_gain>
@@ -53,8 +53,8 @@
                 <odometryTopic>/vector/feedback/wheel_odometry</odometryTopic>
                 <odometryFrame>odom</odometryFrame>
-                <odometryRate>30.0</odometryRate>
+                <odometryRate>100.0</odometryRate>
                 <robotBaseFrame>base_link</robotBaseFrame>
                 <publishOdometryTf>0</publishOdometryTf>
-                <yaw_velocity_p_gain>100.0</yaw_velocity_p_gain>
+                <yaw_velocity_p_gain>500.0</yaw_velocity_p_gain>
                 <x_velocity_p_gain>10000.0</x_velocity_p_gain>
                 <y_velocity_p_gain>10000.0</y_velocity_p_gain>

File: vector_common/vector_description/urdf/vector_components/vector_base.urdf.xacro (robot description, xacro)
@@ -27,7 +27,4 @@
         <!-- Base link is the center of the robot's chassis between the motors projected on the ground -->
         <link name="base_link"/>
-        <gazebo reference="base_link">
-            <mu1>0.0</mu1>
-        </gazebo>
         <joint name="base_chassis_joint" type="fixed">
             <origin xyz="0 0 ${wheel_radius}" rpy="0 0 0" />
@@ -36,11 +33,11 @@
         </joint>
         <link name="base_chassis_link">
-			<inertial>
-				<mass value="44.2877" />
-				<origin xyz="-0.009506 -0.013039 0.032319" />
-				<inertia ixx="0.000165"  ixy="0" ixz="0"
-                         iyx="0"  iyy="0.000559" iyz="0"
-                         izx="0" izy="0" izz="0.000714" />
-			</inertial>
+	    <inertial>
+		    <mass value="101.561195" />
+		    <origin xyz="-0.000710 -0.000186 0.03813" rpy="0 0 0"/>
+		    <inertia ixx="3.126061"  ixy="-0.032687" ixz="-0.086662"
+                         iyx="-0.032687" iyy="13.356772" iyz="0.000468"
+                         izx="-0.086662" izy="0.000468"  izz="15.218700" />
+	    </inertial>
             <collision>
 				<geometry>
@@ -56,5 +53,9 @@
 		</link>
         <gazebo reference="base_chassis_link">
-            <mu1>0.0</mu1>
+			<mu1 value="0.1"/>
+			<mu2 value="0.1"/>
+			<kp value="10000000.0" />
+			<kd value="1.0" />
+			<fdir1 value="1 0 0"/>
         </gazebo>
         <joint name="payload_plate_joint" type="fixed">
@@ -83,4 +84,11 @@
 			</visual>
 		</link>
+        <gazebo reference="payload_plate_joint">
+			<mu1 value="0.1"/>
+			<mu2 value="0.1"/>
+			<kp value="10000000.0" />
+			<kd value="1.0" />
+			<fdir1 value="1 0 0"/>
+        </gazebo>
     </xacro:macro>
 </robot>

Commit message: adding safety laser configuration

File: vector_common/vector_description/urdf/accessories.urdf.xacro (robot description, xacro)
@@ -23,4 +23,5 @@
 <robot name="vector_accessories" xmlns:xacro="http://ros.org/wiki/xacro">
     <xacro:include filename="$(find vector_description)/urdf/sensors/sick_tim.urdf.xacro"/>
+    <xacro:include filename="$(find vector_description)/urdf/sensors/hokuyo_uam_05lp.urdf.xacro"/>
     <xacro:property name="M_PI" value="3.14159"/>
     <xacro:macro name="vector_accessories">
@@ -45,10 +46,20 @@
             </plugin>
         </gazebo>
-        <xacro:sick_tim laser_prefix="front" parent="base_chassis_link">
-            <origin xyz="$(optenv LASER1_XYZ 0.3075 0 0.1439106)" rpy="$(optenv LASER1_RPY 3.14159 0 0)" />
-        </xacro:sick_tim>
-        <xacro:sick_tim laser_prefix="rear" parent="base_chassis_link">
-            <origin xyz="$(optenv LASER2_XYZ -0.3075 0 0.1439106)" rpy="$(optenv LASER2_RPY 3.14159 0 3.14159)" />
-        </xacro:sick_tim>
+        <xacro:unless value="$(optenv VECTOR_HAS_SAFETY_LASERS false)">
+            <xacro:sick_tim laser_prefix="front" parent="base_chassis_link">
+                <origin xyz="0.3075 0 0.1439106" rpy="3.14159 0 0" />
+            </xacro:sick_tim>
+            <xacro:sick_tim laser_prefix="rear" parent="base_chassis_link">
+                <origin xyz="-0.3075 0 0.1439106" rpy="3.14159 0 3.14159" />
+            </xacro:sick_tim>
+        </xacro:unless>
+        <xacro:if value="$(optenv VECTOR_HAS_SAFETY_LASERS false)">
+            <xacro:hokuyo_uam_05lp laser_prefix="front" parent="base_chassis_link">
+                <origin xyz="0.252995 0.192212 0.137128" rpy="${M_PI} 0 ${M_PI/4}"/>
+            </xacro:hokuyo_uam_05lp>
+            <xacro:hokuyo_uam_05lp laser_prefix="rear" parent="base_chassis_link">
+                <origin xyz="-0.252995 -0.192212 0.137128" rpy="${M_PI} 0 ${5*M_PI/4}" />
+            </xacro:hokuyo_uam_05lp>
+        </xacro:if>
     </xacro:macro>
 </robot>
